File: BMS2.kicad_pcb (KiCad board)
At the start: 4 copper layers, 139 x 36 mm, 169 parts, among them J1 XT30PW-M, J2 XT30PW-F, J3 B12B-XH-A(LF)(SN), J4 B13B-XH-A(LF)(SN), J5 10129378-903004BLF, J6 B4B-PH-K-S(LF)(SN), J7 B2B-PH-K-S(LF)(SN), J8 B2B-PH-K-S(LF)(SN), Q1 RD3S100CNTL1, Q2 AO3401A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

Commit message: Add files via upload
Parts:
- removed the G*** at (79.5, 83.2)
